File: PowerSupplyProject.kicad_pcb (KiCad board)
At the start: 2 copper layers, 30.5 x 53 mm, 17 parts, among them J1 Conn_01x02_Pin, J2 Conn_01x02_Pin, J3 Conn_01x03_Pin, J4 Conn_01x03_Pin, J5 Screw_Terminal_01x02, J7 Screw_Terminal_01x02, J8 Barrel_Jack_Switch, SW1 EG1218, U1 LM7805, U2 LM317

Commit message: fix the route
Routing:
- net /PWR_output: track 0.44 -> 79.3 mm
- net /12V: track 0.36 -> 56.3 mm
- net /3.3V: track 0.00 -> 51.4 mm, vias 0 -> 1
- net /5V: track 0.00 -> 47.6 mm
- net /3V: track 0.00 -> 17.8 mm
- net /PWR_input: track 2.04 -> 15.8 mm
- net Net-(U1-VO): track 0.00 -> 10.6 mm
- net Net-(U2-ADJ): track 0.14 -> 9.56 mm
- net Net-(D1-A): track 0.00 -> 7.06 mm

Commit message: route fixed
Routing:
- net /PWR_output: track 79.3 -> 96.2 mm
Changed lines of the file:
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@@
+	)
+	(segment
+		(start 134.5 69.5)
+		(end 137 72)
+		(width 0.35)
+		(layer "F.Cu")
+		(net "/PWR_output")
 	)
 	(segment
@@
 		(start 139 114.5)
 		(end 139 74)
+		(width 0.35)
+		(layer "F.Cu")
+		(net "/PWR_output")
+	)
+	(segment
+		(start 122.682 71.5)
+		(end 122.682 70.318)
+		(width 0.35)
+		(layer "F.Cu")
+		(net "/PWR_output")
+	)
+	(segment
+		(start 123.5 69.5)
+		(end 134.5 69.5)
 		(width 0.35)
 		(layer "F.Cu")
@@
 		(width 0.35)
 		(layer "F.Cu")
+		(net "/PWR_output")
+	)
+	(segment
+		(start 122.682 70.318)
+		(end 123.5 69.5)
+		(width 0.35)
+		(layer "F.Cu")

Commit message: fixed the schematic label and value components
Routing:
- net /PWR_output: track 96.2 -> 50.7 mm
- net GND: track 0.00 -> 1.95 mm
Changed lines of the file:
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@@
+	)
+	(segment
+		(start 119.5 76)
+		(end 117.55 76)
+		(width 0.25)
+		(layer "F.Cu")
+		(net "GND")
 	)
 	(segment
@@
 	)
 	(segment
-		(start 137.5 116)
-		(end 139 114.5)
-		(width 0.35)
-		(layer "F.Cu")
-		(net "/PWR_output")
-	)
-	(segment
 		(start 134.5 69.5)
 		(end 137 72)
 		(width 0.35)
 		(layer "F.Cu")
-		(net "/PWR_output")
-	)
-	(segment
-		(start 139 74)
-		(end 137 72)
-		(width 0.35)
-		(layer "F.Cu")
-		(net "/PWR_output")
-	)
-	(segment
-		(start 139 114.5)
-		(end 139 74)
-		(width 0.35)
-		(layer "F.Cu")

Commit message: fix route based on fixed label
Parts:
- R1, R2: value 330R -> 330
- R3: value 560R -> 560
- U1: value LM7805 -> LM7805_TO220
- U2: value LM317 -> LM317_TO-220
- moved U2 5.18 mm to (121.0, 104.0), turned to 0 degrees
- moved C1 2.75 mm to (119.2, 80.0), turned to 0 degrees
- moved C2 2.75 mm to (119.2, 76.0), turned to 0 degrees
Connections:
- C2 pad 1: Net-(U1-VO) -> /5V
- C3 pad 1: /3V -> /3.3V
- J1 pad 2: /PWR_output -> /PWR_output_top
- J2 pad 2: /PWR_output -> /PWR_output_bot
- J3 pad 2: /PWR_output -> /PWR_output_top
- J4 pad 2: /PWR_output -> /PWR_output_bot
- J5 pad 2: /PWR_output -> /PWR_output_top
- J7 pad 2: /PWR_output -> /PWR_output_bot
- R3 pad 1: /3V -> /3.3V
- U1 pad 3: Net-(U1-VO) -> /5V
- U2 pad 2: /3V -> /3.3V
Routing:
- net /PWR_output: track 50.7 -> 0.00 mm
- net /PWR_output_bot: track 0.00 -> 25.9 mm
- net /PWR_output_top: track 0.00 -> 24.4 mm
- net /3V: track 17.8 -> 0.00 mm
- net /3.3V: track 51.4 -> 64.7 mm
- net Net-(U1-VO): track 10.6 -> 0.00 mm
- net Net-(U2-ADJ): track 9.56 -> 17.4 mm, vias 0 -> 1
- net /5V: track 47.6 -> 50.1 mm
- net GND: track 1.95 -> 0.00 mm
- net /12V: track 56.3 -> 54.9 mm
